File: eagle/project/simple_clock.brd (EAGLE design)
At the start: 75.5 x 70.7 mm, 10 parts, among them U1 STM32F103C8T6, U2 MAX7219CNG, U3 AMS1117_50_REG

Commit message: updated firmware
Parts:
- moved C1 0.38 mm to (77.9, 24.1), turned to 180 degrees
Routing:
- net N$11: track 76.3 -> 91.9 mm, vias 3 -> 2
- net N$4: track 29.7 -> 18.0 mm, vias 2 -> 1
- net N$15: track 31.6 -> 42.2 mm, vias 2 -> 1
- net N$17: track 65.8 -> 72.9 mm, vias 6 -> 4
- net N$18: track 62.8 -> 58.9 mm, vias 4 -> 2
- net GND: track 199.6 -> 203.1 mm
- net N$16: track 49.6 -> 46.7 mm
- net +5V: track 74.7 -> 76.3 mm, vias 2 -> 1
- net N$14: track 94.2 -> 95.3 mm, vias 3 -> 2
- net N$12: track 61.0 -> 60.0 mm, vias 4 -> 3
- net N$25: track 49.6 -> 50.4 mm, vias 3 -> 2
- net N$19: track 28.6 -> 28.1 mm, vias 1 -> 0
- net N$23: vias 0 -> 1
- net N$24: vias 0 -> 1
